File: tests/kicad8/warning-project/logic.kicad_sch (KiCad schematic)
At the start: 5 parts, among them U1 74LS04, U2 74AHC1G126, U4 74AHC1G126

Commit message: [PCBNew][DRC] Implemented CLI version
Parts:
- U1: footprint (none) -> Package_SO:SOIC-14_3.9x8.7mm_P1.27mm
- U2, U4: footprint (none) -> Package_TO_SOT_SMD:SOT-23-5
Connections:
- net at U1.2: now also U1.4
- net at U2.4: now also U1.6
- no-connect marks 6 -> 2

Commit message: [EEschema][ERC] Implemented kicad-cli JSON parser
Connections:
- net at U1.2: no longer U1.4
- no-connect marks 2 -> 4
Changed lines of the file:
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@@
+	)
+	(no_connect
+		(at 168.91 82.55)
 	)
 	(no_connect
@@
 		(at 214.63 95.25)
 	)
+	(no_connect
+		(at 171.45 82.55)
+	)
 	(wire
 		(pts
@@
 		(pts
 			(xy 195.58 58.42) (xy 195.58 60.96)
-		)
-		(stroke
-			(width 0)
-			(type solid)
-		)
-	)
-	(wire
-		(pts
-			(xy 168.91 82.55) (xy 171.45 82.55)
 		)
 		(stroke
@@
 		)
 		(instances
-			(project "fail-project"
+			(project "warning-project"
 				(path "/87c78429-be2b-40ed-8d3b-56cb9666a56f/00000000-0000-0000-0000-00005ca75bc1"
 					(reference "R1")
@@
 		)
 		(instances
-			(project "fail-project"
+			(project "warning-project"
 				(path "/87c78429-be2b-40ed-8d3b-56cb9666a56f/00000000-0000-0000-0000-00005ca75bc1"
 					(reference "C2")
@@
 		)
 		(instances
-			(project "fail-project"
+			(project "warning-project"
 				(path "/87c78429-be2b-40ed-8d3b-56cb9666a56f/00000000-0000-0000-0000-00005ca75bc1"
 					(reference "#PWR03")
@@
 		)
 		(instances
-			(project "fail-project"
+			(project "warning-project"
 				(path "/87c78429-be2b-40ed-8d3b-56cb9666a56f/00000000-0000-0000-0000-00005ca75bc1"
 					(reference "U1")
@@
 		)
 		(instances
-			(project "fail-project"
+			(project "warning-project"
 				(path "/87c78429-be2b-40ed-8d3b-56cb9666a56f/00000000-0000-0000-0000-00005ca75bc1"
 					(reference "U1")
@@
 		)
 		(instances
-			(project "fail-project"
+			(project "warning-project"
 				(path "/87c78429-be2b-40ed-8d3b-56cb9666a56f/00000000-0000-0000-0000-00005ca75bc1"
 					(reference "#PWR05")
@@
 		)
 		(instances
-			(project "fail-project"
+			(project "warning-project"
 				(path "/87c78429-be2b-40ed-8d3b-56cb9666a56f/00000000-0000-0000-0000-00005ca75bc1"
 					(reference "#PWR04")
@@
 		)
 		(instances
-			(project "fail-project"
+			(project "warning-project"
 				(path "/87c78429-be2b-40ed-8d3b-56cb9666a56f/00000000-0000-0000-0000-00005ca75bc1"
 					(reference "#PWR011")
@@
 		)
 		(instances
-			(project "fail-project"
+			(project "warning-project"
 				(path "/87c78429-be2b-40ed-8d3b-56cb9666a56f/00000000-0000-0000-0000-00005ca75bc1"
 					(reference "#PWR0101")
@@
 		)
 		(instances
-			(project "fail-project"
+			(project "warning-project"
 				(path "/87c78429-be2b-40ed-8d3b-56cb9666a56f/00000000-0000-0000-0000-00005ca75bc1"
 					(reference "#PWR06")
@@
 		)
 		(instances
-			(project "fail-project"
+			(project "warning-project"
 				(path "/87c78429-be2b-40ed-8d3b-56cb9666a56f/00000000-0000-0000-0000-00005ca75bc1"
 					(reference "U2")
@@
 		)
 		(instances
-			(project "fail-project"
+			(project "warning-project"
 				(path "/87c78429-be2b-40ed-8d3b-56cb9666a56f/00000000-0000-0000-0000-00005ca75bc1"
 					(reference "#PWR0103")
@@
 		)
 		(instances
-			(project "fail-project"
+			(project "warning-project"
 				(path "/87c78429-be2b-40ed-8d3b-56cb9666a56f/00000000-0000-0000-0000-00005ca75bc1"
 					(reference "U1")
@@
 		)
 		(instances
-			(project "fail-project"
+			(project "warning-project"
 				(path "/87c78429-be2b-40ed-8d3b-56cb9666a56f/00000000-0000-0000-0000-00005ca75bc1"
 					(reference "U4")
@@
 		)
 		(instances
-			(project "fail-project"
+			(project "warning-project"
 				(path "/87c78429-be2b-40ed-8d3b-56cb9666a56f/00000000-0000-0000-0000-00005ca75bc1"
 					(reference "#PWR09")
@@
 		)
 		(instances
-			(project "fail-project"
+			(project "warning-project"
 				(path "/87c78429-be2b-40ed-8d3b-56cb9666a56f/00000000-0000-0000-0000-00005ca75bc1"
 					(reference "U1")
@@
 		)
 		(instances
-			(project "fail-project"
+			(project "warning-project"
 				(path "/87c78429-be2b-40ed-8d3b-56cb9666a56f/00000000-0000-0000-0000-00005ca75bc1"
 					(reference "#PWR07")
@@
 		)
 		(instances
-			(project "fail-project"
+			(project "warning-project"
 				(path "/87c78429-be2b-40ed-8d3b-56cb9666a56f/00000000-0000-0000-0000-00005ca75bc1"
 					(reference "U1")
@@
 		)
 		(instances
-			(project "fail-project"
+			(project "warning-project"
 				(path "/87c78429-be2b-40ed-8d3b-56cb9666a56f/00000000-0000-0000-0000-00005ca75bc1"
 					(reference "U1")
@@
 		)
 		(instances
-			(project "fail-project"
+			(project "warning-project"
 				(path "/87c78429-be2b-40ed-8d3b-56cb9666a56f/00000000-0000-0000-0000-00005ca75bc1"
 					(reference "#PWR010")
@@
 		)
 		(instances
-			(project "fail-project"
+			(project "warning-project"
 				(path "/87c78429-be2b-40ed-8d3b-56cb9666a56f/00000000-0000-0000-0000-00005ca75bc1"
 					(reference "U1")
@@
 		)
 		(instances
-			(project "fail-project"
+			(project "warning-project"
 				(path "/87c78429-be2b-40ed-8d3b-56cb9666a56f/00000000-0000-0000-0000-00005ca75bc1"
 					(reference "#PWR0102")
@@
 		)
 		(instances
-			(project "fail-project"
+			(project "warning-project"
 				(path "/87c78429-be2b-40ed-8d3b-56cb9666a56f/00000000-0000-0000-0000-00005ca75bc1"
 					(reference "#PWR08")
